File: circuit-mecha-donald.kicad_pcb (KiCad board)
At the start: 2 copper layers, 111 x 86 mm, 43 parts, among them J1 ST-LINK, J10 MD6, J11 ENC1, J12 ENC2, J13 ENC3, J14 ENC4, J15 ENC5, J16 ENC6, J2 CAN, J3 UART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

Commit message: feature: CANコネクタを追加。
Parts:
- added J17: CAN2, Connector_JST:JST_XA_S04B-XASK-1N-BN_1x04_P2.50mm_Horizontal, F.Cu at (201.0, 85.0)
- J2: value CAN -> CAN1
- moved J1 7.00 mm to (194.0, 84.8)
Routing:
- net CAN_P: track 21.4 -> 40.0 mm
- net CAN_N: track 23.0 -> 41.6 mm
- net +5V: track 306.8 -> 323.9 mm
- net +3.3V: track 360.3 -> 353.3 mm
- net SWCLK: track 42.9 -> 36.2 mm, vias 2 -> 1
- net NRST: track 119.4 -> 114.8 mm
- net SWDIO: track 42.8 -> 38.2 mm
- net SWO: track 54.8 -> 50.8 mm
- net GND: track 32.7 -> 34.0 mm, vias 168 -> 166
